File: KiCad_Eurocard_0/KiCad_Eurocard_0.kicad_sch (KiCad schematic)
At the start: 62 parts, among them IC1 ERA-1SM+, IC2 ADF4351BCPZ, IC3 ERA-1SM+, IC4 AD9959BCPZ, IC5 ADF4351BCPZ, J1 Conn_Coaxial, J2 Conn_Coaxial, J3 Conn_Coaxial, J4 Conn_Coaxial, J5 Conn_Coaxial, J6 Conn_Coaxial, J7 Conn_Coaxial, J8 Conn_Coaxial

Commit message: Updated R + C values/made pretty, ADF4351 still work in progress
need to go off datasheet for ADF4351 as well as the eval board (google ADF4351 Eval board and it will give you an example of the board in use.)
Parts:
- removed C10, C7, C8, C9: C, symbol Device:C
- removed IC1, IC3: ERA-1SM+, ERA-1SM+:ERA1SM, symbol ERA-1SM+:ERA-1SM+
- removed IC2: ADF4351BCPZ, ADF4351BPCZ:QFN50P500X500X100-33N, symbol ADF4351BCPZ:ADF4351BCPZ
- added A1, A2: ERA-1SM+, ERA-1SM+:ERA1SM, symbol ERA-1SM+:ERA-1SM+
- added A3: Arduino_Nano_ESP32, Module:Arduino_Nano, symbol MCU_Module:Arduino_Nano_ESP32
- added C12, C13: 300pF, Capacitor_SMD:C_0402_1005Metric, symbol Device:C
- added C14: 1.78nF, symbol Device:C
- added C15: 100pF, symbol Device:C
- added C16: 10nF, symbol Device:C
- added C17: 1uF, symbol Device:C
- added R37: 90.9 Ohms, symbol Device:R
- added R38: 251 Ohms, symbol Device:R
- C1, C2: value C -> 300pF
- C11: value 10 pF -> 47.3nF
- C3: value C -> 1uF; footprint Capacitor_SMD:C_0402_1005Metric -> (none)
- C4: value C -> 10nF; footprint Capacitor_SMD:C_0402_1005Metric -> (none)
- C5: value C -> 100pF; footprint Capacitor_SMD:C_0402_1005Metric -> (none)
- C6: value C -> 208pF; footprint Capacitor_SMD:C_0402_1005Metric -> (none)
- R1: value R -> 90.9 Ohms; footprint Resistor_SMD:R_0402_1005Metric -> (none)
- R2: value 20.5 Ohm -> 116.1 Ohms
- R3: value 150 Ohm -> 52.8 Ohms
- R36: value R -> 5.10k Ohms
- R4: value 150 Ohm -> 116.1 Ohms
- R5: value R -> 1.57k Ohms; footprint Resistor_SMD:R_0402_1005Metric -> (none)
- R6, R8: value R -> 178.5 Ohms
- R7: value R -> 30.4 Ohms
Connections:
- net 3.3V: now also IC5.16 (VVCO_2)
- net GND: now also C11.2, C3.2, C4.2, C5.2, C6.2, IC5.11 (AGNDVCO_2), IC5.18 (AGNDVCO_3), IC5.21 (AGNDVCO), IC5.31 (SDGND), IC5.8 (CPGND), R2.2, A1.2 (GND_1), A1.4 (GND_2), A2.2 (GND_1), A2.4 (GND_2), C14.2, C15.2, C16.2, C17.2; no longer C2.1, C6.1, R3.2
- net S1 Port 1: now also R24.1, R26.2, S1.6 (_PORT_1)
- net REF IN: now reaches R25.1, R26.1
- net REF IN: now also IC5.24 (VREF)
- net at R6.1, R7.2: now also C2.1; no longer C5.1
- net at IC5.29 (REFIN): no longer C11.1
- net A1 OUT: now reaches R4.1, S1.1 (SUM_PORT)
- net A1 OUT: now also R3.1; no longer R2.1
- net 7V: now reaches C4.1
- net 7V: now also C3.1, C5.1, R1.2, C15.1, C16.1, C17.1, R37.2
- net S1 Port 5: now reaches S1.3 (PORT_5)
- net S1 Port 5: now also C1.2; no longer C4.2
- net A2 OUT: now reaches R7.1, R8.1, S2.1 (SUM_PORT)
- net ADF4351 Loop: now reaches IC5.20 (VTUNE)
- net ADF4351 Loop: now also R5.1, C14.1, R38.2
- net at IC5.22 (RSET): now also R36.1
- net Lock Detect Out: now reaches IC5.30 (MUXOUT)
- net Chip Enable: now reaches IC5.4 (CE)
- net at IC5.7 (CPOUT): now also C6.1, R5.2
- net at R1.1: now also C2.2, A2.1 (RF_IN); no longer C3.2
- net at C1.1: now also A2.3 (RF_-_OUT_AND_DC_-_IN)
- removed net +VDC: C2.2, C6.2, R1.2, R5.2
- new net: A3.29 (GND), A3.4 (GND)
- new net: A1.1 (RF_IN), C13.2, R37.1
- new net: A1.3 (RF_-_OUT_AND_DC_-_IN), C12.1
- new net: C11.1, R38.1
- new net: C13.1, R2.1, R3.2
- new net 100MHz OXCO: C12.2
- no-connect marks 0 -> 1
Other:
- moved on the sheet: IC4, IC5, R24, R25, R26, R6, R7, R8, S1, S2

Commit message: ADF4351 Microcontroller Connecs. Done
- Added Microcontroller and connections to the ADF4351
- Started parameters note sheet
- Need to double check power is sufficient for circuit (hopefully, we can just use the 5V USB to power everything?)
- Need to make schematic look pretty as well/be more organized/labeled
Parts:
- removed A3: Arduino_Nano_ESP32, Module:Arduino_Nano, symbol MCU_Module:Arduino_Nano_ESP32
- removed IC4: AD9959BCPZ, QFN50P800X800X100-57N-D, symbol AD9959BCPZ:AD9959BCPZ
- added C10, C19, C21, C23, C25, C39, C42, C48, C50, C52, C8: 10pF, symbol Device:C
- added C18, C20, C22, C24, C38, C40, C41, C43, C46, C47, C49, C51, C7, C9: 0.1uF, symbol Device:C
- added C26: 100nF, symbol Device:C
- added C30: 22uF, symbol Device:C
- added C31, C32, C33, C34, C35, C37: 1uF, symbol Device:C
- added C36: 1nF, symbol Device:C
- added C44, C45: 12pF, symbol Device:C
- added D1, D4, D5: LED, symbol Device:LED
- added D2, D3: BZX84Cxx, Package_TO_SOT_SMD:SOT-23, symbol Diode:BZX84Cxx
- added IC1: ADP3334ARZ, SOIC127P600X175-8N, symbol ADP3334ARZ:ADP3334ARZ
- added IC2: AD9959BCPZ, QFN50P800X800X100-57N-D, symbol AD9959BCPZ:AD9959BCPZ
- added J9: USB_B_Mini, symbol Connector:USB_B_Mini
- added R39: 1k Ohm, symbol Device:R
- added R40, R45, R46: 2.2k Ohm, symbol Device:R
- added R41: 78.7k Ohm, symbol Device:R
- added R42: 140k Ohm, symbol Device:R
- added R43, R44: 100k Ohm, symbol Device:R
- added R47, R48, R49, R50: 10k Ohm, symbol Device:R
- added R51: 100 Ohm, symbol Device:R
- added SW1, SW2: SW_DIP_x01, symbol Switch:SW_DIP_x01
- added U1, U2: ADP150ACBZ-2.85R7, ADP150:CB_4_3_ADI, symbol ADP150:ADP150ACBZ-2.85R7
- added U3: CY7C68013A-56LTX, Package_DFN_QFN:QFN-56-1EP_8x8mm_P0.5mm_EP4.5x5.2mm_ThermalVias_TopTented, symbol MCU_Cypress:CY7C68013A-56LTX
- added U4: 24LC64, symbol Memory_EEPROM:24LC64
- added Y1: ECS-240-12-20A-TR, ECS2401220ATR, symbol ECS-240-12-20A-TR:ECS-240-12-20A-TR
Connections:
- net 3.3V is gone; now on net AVDD (3.3V): IC5.10 (AVDD), IC5.16 (VVCO_2), IC5.17 (VVCO), IC5.28 (DVDD), IC5.32 (SDVDD), IC5.6 (VP)
- net Chip Enable: now also R50.1
- net GND: now also IC5.33 (EP), C10.2, C18.2, C19.2, C20.2, C21.2, C22.2, C23.2, C24.2, C25.2, C30.2, C31.2, C32.2, C33.2, C34.2, C35.2, C37.2, C38.2, C39.2, C40.2, C41.2, C42.2, C43.2, C44.2, C45.2, C46.2, C47.2, C48.2, C49.2, C50.2, C51.2, C52.2, C7.2, C8.2, C9.2, D1.1 (K), D2.1 (A), D4.1 (K), D5.1 (K), IC1.1 (GND), IC1.2 (SD), J9.4 (ID), J9.5 (GND), J9.6 (Shield), R41.1, R47.2, R48.2, R49.2, U1.B2 (GND), U2.B2 (GND), U3.1 (RDY0/SLRD), U3.10 (AGND), U3.12 (GND), U3.14 (RESERVED), U3.2 (RDY1/SLWR), U3.26 (GND), U3.28 (GND), U3.41 (GND), U3.53 (GND), U3.56 (GND), U3.6 (AGND), U4.2 (A1), U4.3 (A2), U4.4 (GND), U4.7 (WP)
- net REF IN: now also IC5.29 (REFIN), C26.2; no longer IC5.24 (VREF), R25.1, R26.1
- net CLK: now reaches IC5.1 (CLK)
- net CLK: now also R47.1, U3.34 (PA1/~{INT1})
- net Temp: now reaches IC5.19 (TEMP)
- net Temp: now also C51.1, C52.1
- net Data: now reaches IC5.2 (DATA)
- net Data: now also R48.1
- net VCom: now reaches IC5.23 (VCOM)
- net VCom: now also C49.1, C50.1
- net at IC5.25 (LD): now also R51.1
- net AVDD (3.3V): now reaches IC5.26 (PDBRF)
- net AVDD (3.3V): now also C10.1, C18.1, C19.1, C20.1, C21.1, C22.1, C23.1, C24.1, C25.1, C34.1, C7.1, C8.1, C9.1, R39.1, R50.2, U2.A2 (VOUT)
- net Load Enable: now reaches IC5.3 (LE)
- net Load Enable: now also R49.1, U3.33 (PA0/~{INT0})
- net Lock Detect Out renamed MUXOUT
- net MUXOUT: now also U3.18 (PB0/FD0)
- new net: C36.1, IC1.7 (FB), R41.2, R42.1
- new net: C30.1, C31.1, C32.1, D3.3 (K), SW1.2, U1.A1 (VIN), U1.B1 (EN), U2.A1 (VIN), U2.B1 (EN)
- new net: C26.1, R25.1, R26.1
- new net: D1.2 (A), R39.2
- new net: J9.2 (D-), U3.9 (D-)
- new net: J9.3 (D+), U3.8 (D+)
- new net: D4.2 (A), R40.2
- new net: D3.1 (A), SW2.2
- new net: D5.2 (A), R51.2
- new net 3V3_USB: C36.2, C37.1, C38.1, C39.1, C42.1, C43.1, C46.1, IC1.5 (OUT_1), IC1.6 (OUT_2), R42.2, R43.1, R44.1, R45.1, R46.1, U3.11 (VCC), U3.17 (VCC), U3.27 (VCC), U3.3 (AVCC), U3.32 (VCC), U3.43 (VCC), U3.55 (VCC), U3.7 (AVCC), U4.1 (A0), U4.8 (VCC)
- new net 5V_USB: C35.1, IC1.3 (IN_1), IC1.4 (IN_2), J9.1 (VBUS), R40.1, SW2.1
- new net DATA: U3.35 (PA2/SLOE)
- new net External 5.5V Source: D2.3 (K), SW1.1
- new net RESET: C41.1, R43.2, U3.42 (~{RESET})
- new net SCL: R45.2, U3.15 (SCL), U4.6 (SCL)
- new net SDA: R46.2, U3.16 (SDA), U4.5 (SDA)
- new net VRef: C47.1, C48.1, IC5.24 (VREF)
- new net Vout: C33.1, U1.A2 (VOUT)
- new net WAKEUP: C40.1, R44.2, U3.44 (WAKEUP)
- new net XTALIN: C44.1, U3.5 (XTALIN), Y1.1
- new net XTALOUT: C45.1, U3.4 (XTALOUT), Y1.2
Other:
- moved on the sheet: A1, A2, C1, C11, C12, C13, C14, C15, C16, C17, C2, C3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

Commit message: added Balun for ADF4351 output
added Balun for ADF4351 0utput. Just need 5v to 7v converter, all footprints, and to wire up DDS.
Parts:
- added C27, C28: 5.6 pF, symbol Device:C
- added C29: 120 pF, symbol Device:C
- added L1: 180 nH, symbol Device:L
- added L2, L3: 51 nH, symbol Device:L
- added R52: 50 Ohms, symbol Device:R
Connections:
- net GND: now also C28.2, R52.1
- net Vout: now also L1.1, L2.1
- net at C13.2, R37.1: now also A1.3 (RF_-_OUT_AND_DC_-_IN); no longer A1.1 (RF_IN)
- net at C12.1: now also A1.1 (RF_IN); no longer A1.3 (RF_-_OUT_AND_DC_-_IN)
- net RFoutA+: now reaches IC5.12 (RFOUTA+)
- net RFoutA+: now also C27.1, L2.2
- net RFoutA-: now reaches IC5.13 (RFOUTA-)
- net RFoutA-: now also C28.1, L1.2, L3.2
- net at C1.1: now also A2.1 (RF_IN); no longer A2.3 (RF_-_OUT_AND_DC_-_IN)
- net at C2.2, R1.1: now also A2.3 (RF_-_OUT_AND_DC_-_IN); no longer A2.1 (RF_IN)
- new net: C27.2, C29.1, L3.1
- new net: C29.2, R52.2
- no-connect marks 1 -> 3
Other:
- moved on the sheet: A1, A2

Commit message: Adjusted layout tbh to make look prettier
-Changed USB power circuits into one power supply
Parts:
- added L4, L5: 470 nH, symbol Device:L
- added R53: 1.91k Ohm, Resistor_SMD:R_0402_1005Metric, symbol Device:R
- renumbered IC5 to IC1, U3 to IC2
Connections:
- net AVDD (3.3V): now also IC2.49 (DVDD_I/O)
- net GND: now also IC2.10 (AGND_2), IC2.12 (AGND_3), IC2.16 (AGND_4), IC2.18 (AGND_5), IC2.20 (AGND_6), IC2.25 (AGND_7), IC2.28 (AGND_8), IC2.32 (AGND_9), IC2.34 (AGND_10), IC2.38 (AGND_11), IC2.44 (DGND_1), IC2.56 (DGND_2), IC2.57 (GND), IC2.6 (AGND_1), R53.1
- net at A1.3 (RF_-_OUT_AND_DC_-_IN), C13.2: now also L4.2; no longer R37.1
- net 300MHz Output: now reaches C29.2, R52.2
- net at IC2.17 (DAC_RSET): now also R53.2
- net 1.8V Source: now reaches IC2.45 (DVDD_1)
- net 1.8V Source: now also IC2.55 (DVDD_2)
- net at A2.3 (RF_-_OUT_AND_DC_-_IN), C2.2: now also L5.2; no longer R1.1
- net 5V_USB renamed VBus
- net CLK renamed CLK IN
- net Chip Enable renamed Chip Enable IN
- net DATA renamed DATA OUT
- net Data renamed Data IN
- net Load Enable renamed Load Enable IN
- net MUXOUT: no longer names the net of IC1.30 (MUXOUT)
- net MUXOUT: no longer IC2.18 (PB0/FD0)
- net Vout renamed Vout (3.3V)
- new net: L4.1, R37.1
- new net: L5.1, R1.1
- no-connect marks 3 -> 4
Other:
- moved on the sheet: C10, C11, C14, C18, C19, C20, C21, C22, C23, C24, C25, C26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
