File: KiCad_Eurocard_0/KiCad_Eurocard_0.kicad_sch (KiCad schematic)
At the start: 138 parts, among them IC1 ADF4351BCPZ, IC1 ADP3334ARZ, IC2 AD9959BCPZ, IC2 CY7C68013A-56LTX, J1 Conn_Coaxial, J2 Conn_Coaxial, J3 Conn_Coaxial, J4 Conn_Coaxial, J5 Conn_Coaxial, J6 Conn_Coaxial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

Commit message: Test Change
Test Change
Parts:
- removed C27, C28: 5.6 pF, symbol Device:C
- removed C29: 120 pF, symbol Device:C
- removed L1: 180 nH, symbol Device:L
- removed L2, L3: 51 nH, symbol Device:L
- added C53, C56: 1 nF, symbol Device:C
- added R54: 33 Ohm, symbol Device:R
- added R55, R56: 50 Ohms, symbol Device:R
- R52: value 50 Ohms -> 33 Ohm
Connections:
- net 1.8V Source: now also IC2.11 (AVDD_3), IC2.15 (AVDD_4), IC2.19 (AVDD_5), IC2.21 (AVDD_6), IC2.26 (AVDD_7), IC2.31 (AVDD_8), IC2.33 (AVDD_9), IC2.37 (AVDD_10), IC2.39 (AVDD_11), IC2.5 (AVDD_1), IC2.7 (AVDD_2)
- net GND: now also R55.1, R56.1; no longer R52.1
- net RFoutA+: now also C53.1
- net RFoutA-: now also C56.1
- net 300MHz Output: no longer names the net of R52.2
- new net: C53.2, R52.1, R56.2
- new net: C56.2, R54.1, R55.2

Commit message: AVery test
Avery Access Test
Connections:
- net 1.8V Source: no longer IC2.45 (DVDD_1)
Changed lines of the file:
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@@
 	(global_label "1.8V Source"
 		(shape input)
-		(at 346.71 256.54 0)
+		(at 347.98 256.54 0)
 		(fields_autoplaced yes)
 		(effects
@@
 		)
 		(property "Intersheetrefs" "${INTERSHEET_REFS}"
-			(at 361.2461 256.54 0)
+			(at 362.5161 256.54 0)
 			(effects
 				(font
